Commit message: px4

File: urdf/px4.urdf.xacro (robot description, xacro)
@@ -1,533 +1,133 @@
-<?xml version="1.0"?>
-<robot name="px4_drone" xmlns:xacro="http://www.ros.org/wiki/xacro">
-  <!-- Properties -->
-  <xacro:property name="namespace" value="" />
-  <xacro:property name="rotor_velocity_slowdown_sim" value="10" />
-  <xacro:property name="mesh_file" value="package://rotors_description/meshes/firefly.dae" />
-  <xacro:property name="mesh_scale" value="1 1 1"/>
-  <xacro:property name="mass" value="1.5" />
-  <xacro:property name="body_width" value="0.47" />
-  <xacro:property name="body_height" value="0.11" />
-  <xacro:property name="mass_rotor" value="0.005" />
-  <xacro:property name="radius_rotor" value="0.128" />
-  <xacro:property name="motor_constant" value="8.54858e-06" />
-  <xacro:property name="moment_constant" value="0.016" />
-  <xacro:property name="time_constant_up" value="0.0125" />
-  <xacro:property name="time_constant_down" value="0.025" />
-  <xacro:property name="max_rot_velocity" value="838" />
-  <xacro:property name="sin30" value="0.5" />
-  <xacro:property name="cos30" value="0.866025403784" />
-  <xacro:property name="rotor_drag_coefficient" value="8.06428e-05" />
-  <xacro:property name="rolling_moment_coefficient" value="1e-06" />
-  <!-- Drone body -->
-  <link name="base_link">
-    <inertial>
-      <mass value="${mass}" />
-      <origin xyz="0 0 0" rpy="0 0 0" />
-      <inertia ixx="0.0347563" ixy="0.0" ixz="0.0" iyy="0.0458929" iyz="0.0" izz="0.0977" />
-    </inertial>
-    <visual>
-      <origin xyz="0 0 0" rpy="0 0 0" />
-      <geometry>
-        <mesh filename="package://rotors_description/meshes/firefly.dae" scale="${mesh_scale}" />
-      </geometry>
-    </visual>
-    <collision>
-      <origin xyz="0 0 0" rpy="0 0 0" />
-      <geometry>
-        <box size="${body_width} 0.635 ${body_height}" />
-      </geometry>
-    </collision>
-  </link>
-  <!-- Rotors -->
-  <xacro:macro name="vertical_rotor" params="robot_namespace suffix direction motor_constant moment_constant parent mass_rotor radius_rotor time_constant_up time_constant_down max_rot_velocity motor_number rotor_drag_coefficient rolling_moment_coefficient color use_own_mesh mesh prop_scale *origin *inertia">
-    <link name="rotor_${motor_number}">
+    <!-- LIDAR link -->
+    <link name="lidar_link">
+      <pose>0 0 0.15 0 0 0</pose>
       <inertial>
-        <mass value="${mass_rotor}" />
-        <xacro:insert_block name="inertia" />
+        <pose>0 0 0 0 0 0</pose>
+        <mass>0.1</mass>
+        <inertia>
+          <ixx>0.0001</ixx>
+          <ixy>0</ixy>
+          <ixz>0</ixz>
+          <iyy>0.0001</iyy>
+          <iyz>0</iyz>
+          <izz>0.0001</izz>
+        </inertia>
       </inertial>
-      <visual>
+      <visual name="lidar_visual">
+        <pose>0 0 0 0 0 0</pose>
         <geometry>
-          <cylinder length="0.005" radius="${radius_rotor}"/>
+          <cylinder>
+            <radius>0.05</radius>
+            <length>0.1</length>
+          </cylinder>
         </geometry>
-        <material name="${color}">
-          <color rgba="0.2 0.2 0.2 1"/>
+        <material>
+          <ambient>0.2 0.2 0.8 1</ambient>
+          <diffuse>0.2 0.2 0.8 1</diffuse>
         </material>
       </visual>
-      <collision>
+      <collision name="lidar_collision">
+        <pose>0 0 0 0 0 0</pose>
         <geometry>
-          <cylinder length="0.005" radius="${radius_rotor}" />
+          <cylinder>
+            <radius>0.05</radius>
+            <length>0.1</length>
+          </cylinder>
         </geometry>
       </collision>
+      <sensor type="ray" name="hokuyo_sim">
+        <always_on>true</always_on>
+        <update_rate>10.0</update_rate>
+        <ray>
+          <scan>
+            <horizontal>
+              <samples>360</samples>
+              <resolution>1</resolution>
+              <min_angle>-3.14159</min_angle>
+              <max_angle>3.14159</max_angle>
+            </horizontal>
+          </scan>
+          <range>
+            <min>0.1</min>
+            <max>30.0</max>
+            <resolution>0.01</resolution>
+          </range>
+          <noise type="gaussian">
+            <mean>0.0</mean>
+            <stddev>0.01</stddev>
+          </noise>
+        </ray>
+        <plugin name="lidar_plugin" filename="libgazebo_ros_laser.so">
+          <topicName>/scan</topicName>
+          <frameName>lidar_link</frameName>
+        </plugin>
+      </sensor>
     </link>
-    <joint name="rotor_${motor_number}_joint" type="continuous">
-      <xacro:insert_block name="origin" />
-      <axis xyz="0 0 1" />
-      <parent link="${parent}" />
-      <child link="rotor_${motor_number}" />
+    <joint name="base_to_lidar" type="fixed">
+      <parent>base_link</parent>
+      <child>lidar_link</child>
     </joint>
-    <gazebo>
-      <plugin name="${suffix}_motor_model" filename="libgazebo_motor_model.so">
-        <robotNamespace>${robot_namespace}</robotNamespace>
-        <jointName>rotor_${motor_number}_joint</jointName>
-        <linkName>rotor_${motor_number}</linkName>
-        <turningDirection>${direction}</turningDirection>
-        <timeConstantUp>${time_constant_up}</timeConstantUp>
-        <timeConstantDown>${time_constant_down}</timeConstantDown>
-        <maxRotVelocity>${max_rot_velocity}</maxRotVelocity>
-        <motorConstant>${motor_constant}</motorConstant>
-        <momentConstant>${moment_constant}</momentConstant>
-        <commandSubTopic>/gazebo/command/motor_speed</commandSubTopic>
-        <motorNumber>${motor_number}</motorNumber>
-        <rotorDragCoefficient>${rotor_drag_coefficient}</rotorDragCoefficient>
-        <rollingMomentCoefficient>${rolling_moment_coefficient}</rollingMomentCoefficient>
-        <motorSpeedPubTopic>/motor_speed/${motor_number}</motorSpeedPubTopic>
-        <rotorVelocitySlowdownSim>${rotor_velocity_slowdown_sim}</rotorVelocitySlowdownSim>
-      </plugin>
-    </gazebo>
-  </xacro:macro>
-  <!-- Rotor 0 -->
-  <xacro:vertical_rotor
-    robot_namespace="${namespace}"
-    suffix="front_right"
-    direction="ccw"
-    motor_constant="${motor_constant}"
-    moment_constant="${moment_constant}"
-    parent="base_link"
-    mass_rotor="${mass_rotor}"
-    radius_rotor="${radius_rotor}"
-    time_constant_up="${time_constant_up}"
-    time_constant_down="${time_constant_down}"
-    max_rot_velocity="${max_rot_velocity}"
-    motor_number="0"
-    rotor_drag_coefficient="${rotor_drag_coefficient}"
-    rolling_moment_coefficient="${rolling_moment_coefficient}"
-    color="blue"
-    use_own_mesh="false"
-    mesh=""
-    prop_scale="1">
-    <origin xyz="0.13 -0.22 0.023" rpy="0 0 0" />
-    <inertia
-      ixx="0.000001" ixy="0.0" ixz="0.0"
-      iyy="0.000001" iyz="0.0"
-      izz="0.000001" />
-  </xacro:vertical_rotor>
-  <!-- Rotor 1 -->
-  <xacro:vertical_rotor
-    robot_namespace="${namespace}"
-    suffix="back_left"
-    direction="ccw"
-    motor_constant="${motor_constant}"
-    moment_constant="${moment_constant}"
-    parent="base_link"
-    mass_rotor="${mass_rotor}"
-    radius_rotor="${radius_rotor}"
-    time_constant_up="${time_constant_up}"
-    time_constant_down="${time_constant_down}"
-    max_rot_velocity="${max_rot_velocity}"
-    motor_number="1"
-    rotor_drag_coefficient="${rotor_drag_coefficient}"
-    rolling_moment_coefficient="${rolling_moment_coefficient}"
-    color="darkgrey"
-    use_own_mesh="false"
-    mesh=""
-    prop_scale="1">
-    <origin xyz="-0.13 0.2 0.023" rpy="0 0 0" />
-    <inertia
-      ixx="0.000001" ixy="0.0" ixz="0.0"
-      iyy="0.000001" iyz="0.0"
-      izz="0.000001" />
-  </xacro:vertical_rotor>
-  <!-- Rotor 2 -->
-  <xacro:vertical_rotor
-    robot_namespace="${namespace}"
-    suffix="front_left"
-    direction="cw"
-    motor_constant="${motor_constant}"
-    moment_constant="${moment_constant}"
-    parent="base_link"
-    mass_rotor="${mass_rotor}"
-    radius_rotor="${radius_rotor}"
-    time_constant_up="${time_constant_up}"
-    time_constant_down="${time_constant_down}"
-    max_rot_velocity="${max_rot_velocity}"
-    motor_number="2"
-    rotor_drag_coefficient="${rotor_drag_coefficient}"
-    rolling_moment_coefficient="${rolling_moment_coefficient}"
-    color="blue"
-    use_own_mesh="false"
-    mesh=""
-    prop_scale="1">
-    <origin xyz="0.13 0.22 0.023" rpy="0 0 0" />
-    <inertia
-      ixx="0.000001" ixy="0.0" ixz="0.0"
-      iyy="0.000001" iyz="0.0"
-      izz="0.000001" />
-  </xacro:vertical_rotor>
-  <!-- Rotor 3 -->
-  <xacro:vertical_rotor
-    robot_namespace="${namespace}"
-    suffix="back_right"
-    direction="cw"
-    motor_constant="${motor_constant}"
-    moment_constant="${moment_constant}"
-    parent="base_link"
-    mass_rotor="${mass_rotor}"
-    radius_rotor="${radius_rotor}"
-    time_constant_up="${time_constant_up}"
-    time_constant_down="${time_constant_down}"
-    max_rot_velocity="${max_rot_velocity}"
-    motor_number="3"
-    rotor_drag_coefficient="${rotor_drag_coefficient}"
-    rolling_moment_coefficient="${rolling_moment_coefficient}"
-    color="darkgrey"
-    use_own_mesh="false"
-    mesh=""
-    prop_scale="1">
-    <origin xyz="-0.13 -0.2 0.023" rpy="0 0 0" />
-    <inertia
-      ixx="0.000001" ixy="0.0" ixz="0.0"
-      iyy="0.000001" iyz="0.0"
-      izz="0.000001" />
-  </xacro:vertical_rotor>
-  <!-- IMU link -->
-  <link name="imu_link">
-    <inertial>
-      <inertia ixx="0.00001" ixy="0.0" ixz="0.0" iyy="0.00001" iyz="0.0" izz="0.00001" />
-      <mass value="0.015" />
-    </inertial>
-  </link>
-  <joint name="imu_joint" type="fixed">
-    <parent link="base_link" />
-    <child link="imu_link" />
-    <origin xyz="0 0 0" rpy="0 0 0" />
-  </joint>
-  <!-- LIDAR link -->
-  <link name="lidar_link">
-    <inertial>
-      <mass value="0.1"/>
-      <origin xyz="0 0 0" rpy="0 0 0"/>
-      <inertia ixx="0.0001" ixy="0.0" ixz="0.0" iyy="0.0001" iyz="0.0" izz="0.0001"/>
-    </inertial>
-    <visual>
-      <geometry>
-        <cylinder radius="0.05" length="0.05"/>
-      </geometry>
-      <material name="black">
-        <color rgba="0.2 0.2 0.2 1"/>
-      </material>
-    </visual>
-    <collision>
-      <geometry>
-        <cylinder radius="0.05" length="0.05"/>
-      </geometry>
-    </collision>
-  </link>
-  <joint name="lidar_joint" type="fixed">
-    <parent link="base_link"/>
-    <child link="lidar_link"/>
-    <origin xyz="0 0 0.15" rpy="0 0 0"/>
-  </joint>
-  <!-- GPS link -->
-  <link name="gps_link">
-    <inertial>
-      <mass value="0.005"/>
-      <origin xyz="0 0 0" rpy="0 0 0"/>
-      <inertia ixx="0.00001" ixy="0.0" ixz="0.0" iyy="0.00001" iyz="0.0" izz="0.00001"/>
-    </inertial>
-  </link>
-  <joint name="gps_joint" type="fixed">
-    <parent link="base_link"/>
-    <child link="gps_link"/>
-    <origin xyz="-0.05 0 0.08" rpy="0 0 0"/>
-  </joint>
-  <!-- Camera link -->
-  <link name="camera_link">
-    <inertial>
-      <mass value="0.02"/>
-      <origin xyz="0 0 0" rpy="0 0 0"/>
-      <inertia ixx="0.00001" ixy="0.0" ixz="0.0" iyy="0.00001" iyz="0.0" izz="0.00001"/>
-    </inertial>
-    <visual>
-      <geometry>
-        <box size="0.05 0.05 0.05"/>
-      </geometry>
-      <material name="red">
-        <color rgba="0.8 0.2 0.2 1"/>
-      </material>
-    </visual>
-    <collision>
-      <geometry>
-        <box size="0.05 0.05 0.05"/>
-      </geometry>
-    </collision>
-  </link>
-  <joint name="camera_joint" type="fixed">
-    <parent link="base_link"/>
-    <child link="camera_link"/>
-    <origin xyz="0 0 -0.1" rpy="0 1.5708 0"/>
-  </joint>
-  <!-- Landing Gear -->
-  <xacro:macro name="landing_leg" params="name x y">
-    <link name="${name}">
+    <!-- Camera link -->
+    <link name="camera_link">
+      <pose>0 0 -0.1 -1.5708 0 0</pose>
       <inertial>
-        <mass value="0.05"/>
-        <origin xyz="0 0 0" rpy="0 0 0"/>
-        <inertia ixx="0.00001" ixy="0.0" ixz="0.0" iyy="0.00001" iyz="0.0" izz="0.00001"/>
+        <pose>0 0 0 0 0 0</pose>
+        <mass>0.05</mass>
+        <inertia>
+          <ixx>0.00001</ixx>
+          <ixy>0</ixy>
+          <ixz>0</ixz>
+          <iyy>0.00001</iyy>
+          <iyz>0</iyz>
+          <izz>0.00001</izz>
+        </inertia>
       </inertial>
-      <visual>
+      <visual name="camera_visual">
+        <pose>0 0 0 0 0 0</pose>
         <geometry>
-          <cylinder radius="0.01" length="0.15"/>
+          <box>
+            <size>0.05 0.05 0.02</size>
+          </box>
         </geometry>
-        <material name="grey">
-          <color rgba="0.5 0.5 0.5 1"/>
+        <material>
+          <ambient>0.2 0.2 0.8 1</ambient>
+          <diffuse>0.2 0.2 0.8 1</diffuse>
         </material>
       </visual>
-      <collision>
+      <collision name="camera_collision">
+        <pose>0 0 0 0 0 0</pose>
         <geometry>
-          <cylinder radius="0.01" length="0.15"/>
+          <box>
+            <size>0.05 0.05 0.02</size>
+          </box>
         </geometry>
       </collision>
+      <sensor type="camera" name="downward_camera">
+        <always_on>true</always_on>
+        <update_rate>30.0</update_rate>
+        <camera name="head_camera">
+          <horizontal_fov>1.047</horizontal_fov>
+          <image>
+            <width>640</width>
+            <height>480</height>
+            <format>R8G8B8</format>
+          </image>
+          <clip>
+            <near>0.02</near>
+            <far>50.0</far>
+          </clip>
+        </camera>
+        <plugin name="camera_controller" filename="libgazebo_ros_camera.so">
+          <alwaysOn>true</alwaysOn>
+          <updateRate>30.0</updateRate>
+          <cameraName>downward_camera</cameraName>
+          <imageTopicName>image_raw</imageTopicName>
+          <cameraInfoTopicName>camera_info</cameraInfoTopicName>
+          <frameName>camera_link</frameName>
+        </plugin>
+      </sensor>
     </link>
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