Commit message: feat: update

File: urdf/ardupilot.urdf.xacro (robot description, xacro)
@@ -68,5 +68,5 @@
     </link>
     <joint name="base_to_lidar" type="fixed">
-      <parent>iris::base_link</parent>
+      <parent>base_link</parent>
       <child>lidar_link</child>
     </joint>
@@ -132,5 +132,5 @@
     </link>
     <joint name="base_to_camera" type="fixed">
-      <parent>iris::base_link</parent>
+      <parent>base_link</parent>
       <child>camera_link</child>
     </joint>
